Commit message: Added Skids and predefined world

File: description/robot.urdf.xacro (robot description, xacro)
@@ -7,4 +7,11 @@
     <xacro:property name="Iy_body" value="{(1/12)*m1*(0.4*0.4+0.3*0.3)}"/>
     <xacro:property name="Iz_body" value="{(1/12)*m1*(0.4*0.4+0.2*0.2)}"/>
+    <xacro:property name="skid_mass" value="0.1"/> <!-- Mass of each skid -->
+    <xacro:property name="skid_radius" value="0.02"/> <!-- Radius of the skid (capsule) -->
+    <xacro:property name="skid_length" value="0.1"/> <!-- Length of the skid (capsule) -->
+    <!-- Calculate Inertia for a Capsule -->
+    <xacro:property name="inertia_xx" value="${(1/12) * skid_mass * (3 * skid_radius * skid_radius + skid_length * skid_length)}"/>
+    <xacro:property name="inertia_yy" value="${(1/12) * skid_mass * (3 * skid_radius * skid_radius + skid_length * skid_length)}"/>
+    <xacro:property name="inertia_zz" value="${(1/2) * skid_mass * skid_radius * skid_radius}"/>
     <!-- Wheel Inertia (calculated) -->
     <xacro:property name="radius_wheel" value="0.08"/>  <!-- radius of wheel -->
@@ -41,7 +48,7 @@
         </visual>
         <collision>
-            <origin xyz="0.0 0.0 0.06" rpy="0.0 0.0 0.0"/>
+            <origin xyz="0.215 0.0 0.06" rpy="0.0 0.0 0.0"/>
             <geometry>
-                <box size="0.4 0.3 0.2"/>
+                <box size="0.38 0.3 0.2"/>
             </geometry>
         </collision>
@@ -50,11 +57,11 @@
         <parent link="base_link"/>
         <child link="chassis"/>
-        <origin xyz="-0.1 0 0"/>
+        <origin xyz="-0.1 0 0.08"/>
     </joint>
     <!-- LEFT WHEEL -->
     <joint name="left_wheel_joint" type="continuous">
-        <parent link="base_link"/>
+        <parent link="chassis"/>
         <child link="left_wheel"/>
-        <origin xyz="0 0.13 0" rpy="-${pi/2} 0 0"/>
+        <origin xyz="0.1 0.13 0" rpy="-${pi/2} 0 0"/>
         <axis xyz="0 0 1"/>
     </joint>
@@ -67,5 +74,5 @@
         </visual>
         <collision>
-            <origin xyz="0 0.13 0" rpy="-${pi/2} 0 0"/>
+            <origin xyz="0 0 0.01" rpy="0 0 0"/>
             <geometry>
                 <cylinder radius="0.08" length="0.04"/>
@@ -76,7 +83,7 @@
     <!-- RIGHT WHEEL -->
     <joint name="right_wheel_joint" type="continuous">
-        <parent link="base_link"/>
+        <parent link="chassis"/>
         <child link="right_wheel"/>
-        <origin xyz="0 -0.13 0" rpy="${pi/2} 0 0"/>
+        <origin xyz="0.1 -0.13 0" rpy="${pi/2} 0 0"/>
         <axis xyz="0 0 -1"/>
     </joint>
@@ -89,5 +96,5 @@
         </visual>
         <collision>
-            <origin xyz="0 0.15 0" rpy="${pi/2} 0 0"/>
+            <origin xyz="0 0 0.01" rpy="0 0 0"/>
             <geometry>
                 <cylinder radius="0.08" length="0.04"/>
@@ -96,4 +103,42 @@
         <xacro:inertia_wheel />
     </link>
+    <!-- LEFT SKID -->
+    <link name="left_skid">
+        <collision>
+            <origin xyz="0.0 0.0 0.00" rpy="0 0 0"/>
+        <geometry>
+            <cylinder radius="${skid_radius}" length="${skid_length}"/>
+        </geometry>
+        </collision>
+        <inertial>
+            <origin xyz="0.0 0.0 0.00" rpy="0 0 0"/>
+            <mass value="${skid_mass}"/>
+            <inertia ixx="${inertia_xx}" ixy="0.0" ixz="0.0" iyy="${inertia_yy}" iyz="0.0" izz="${inertia_zz}"/>
+        </inertial>
+    </link>
+    <joint name="left_skid_joint" type="fixed">
+        <parent link="chassis"/>
+        <child link="left_skid"/>
+        <origin xyz="0.3 -0.1 -0.03" rpy="0 0 0"/>
+    </joint>
+    <!-- RIGHT SKID -->
+    <link name="right_skid">
+        <collision>
+            <origin xyz="0 0 0.0" rpy="0 0 0"/>
+            <geometry>
+                <cylinder radius="${skid_radius}" length="${skid_length}"/>
+            </geometry>
+        </collision>
+        <inertial>
+            <origin xyz="0 0 0.00" rpy="0 0 0"/>
+            <mass value="${skid_mass}"/>
+            <inertia ixx="${inertia_xx}" ixy="0.0" ixz="0.0" iyy="${inertia_yy}" iyz="0.0" izz="${inertia_zz}"/>
+        </inertial>
+    </link>
+    <joint name="right_skid_joint" type="fixed">
+        <parent link="chassis"/>
+        <child link="right_skid"/>
+        <origin xyz="0.3 0.1 -0.03" rpy="0 0 0"/>
+    </joint>
     <xacro:include filename="$(find lawn_robot_project)/description/robot.gazebo"/>
 </robot>

Commit message: Updated mesh URI's to link to objects more generally

File: description/robot.urdf.xacro (robot description, xacro)
@@ -44,5 +44,6 @@
             <origin xyz="0.025 0.175 -0.050" rpy="0 0 0"/>
             <geometry>
-                <mesh filename="file:///home/user/dev_ws/src/lawn_robot_project/meshes/base.dae" scale="0.001 0.001 0.001"/>
+                <!--<mesh filename="file:///home/user/dev_ws/src/lawn_robot_project/meshes/base.dae" scale="0.001 0.001 0.001"/>-->
+                <mesh filename="package://lawn_robot_project/meshes/base.dae" scale="0.001 0.001 0.001"/>
             </geometry>
         </visual>
@@ -70,5 +71,6 @@
             <origin xyz="-0.08 -0.08 0" rpy="0 0 0"/>
             <geometry>
-                <mesh filename="file:///home/user/dev_ws/src/lawn_robot_project/meshes/wheel.dae" scale="0.001 0.001 0.001"/>
+                <!--<mesh filename="file:///home/user/dev_ws/src/lawn_robot_project/meshes/wheel.dae" scale="0.001 0.001 0.001"/>-->
+                <mesh filename="package://lawn_robot_project/meshes/wheel.dae" scale="0.001 0.001 0.001"/>
             </geometry>
         </visual>
@@ -92,5 +94,6 @@
             <origin xyz="-0.08 -0.08 0" rpy="0 0 0"/>
             <geometry>
-                <mesh filename="file:///home/user/dev_ws/src/lawn_robot_project/meshes/wheel.dae" scale="0.001 0.001 0.001"/>
+                <!--<mesh filename="file:///home/user/dev_ws/src/lawn_robot_project/meshes/wheel.dae" scale="0.001 0.001 0.001"/>-->
+                <mesh filename="package://lawn_robot_project/meshes/wheel.dae" scale="0.001 0.001 0.001"/>
             </geometry>
         </visual>

Commit message: Added Range Sensors, modified World

File: description/robot.urdf.xacro (robot description, xacro)
@@ -144,4 +144,68 @@
         <origin xyz="0.3 0.1 -0.03" rpy="0 0 0"/>
     </joint>
-    <xacro:include filename="$(find lawn_robot_project)/description/robot.gazebo"/>
+  <joint type="fixed" name="scan_joint_left">
+    <origin xyz="0.18 0.08 0.17" rpy="0 0 0"/>
+    <child link="scan_link_left"/>
+    <parent link="base_link"/>
+    <axis xyz="0 1 0" rpy="0 0 0"/>
+  </joint>
+  <link name='scan_link_left'>
+    <inertial>
+      <mass value="1e-5"/>
+      <origin xyz="0 0 0" rpy="0 0 0"/>
+      <inertia
+          ixx="1e-6" ixy="0" ixz="0"
+          iyy="1e-6" iyz="0"
+          izz="1e-6"
+      />
+    </inertial>
+    <collision name='collision'>
+      <origin xyz="0 0 0" rpy="0 0 0"/>
+      <geometry>
+        <box size=".01 .01 .01"/>
+      </geometry>
+    </collision>
+  </link>
+  <gazebo reference="scan_link_left">
+    <selfCollide>false</selfCollide>
+    <mu1 value="0.05" />
+    <mu2 value="0.05" />
+  </gazebo>
+  <joint type="fixed" name="scan_joint_right">
+    <origin xyz="0.18 -0.08 0.17" rpy="0 0 0"/>
+    <child link="scan_link_right"/>
+    <parent link="base_link"/>
+    <axis xyz="0 1 0" rpy="0 0 0"/>
+  </joint>
+  <link name='scan_link_right'>
+    <inertial>
+      <mass value="1e-5"/>
+      <origin xyz="0 0 0" rpy="0 0 0"/>
+      <inertia
+          ixx="1e-6" ixy="0" ixz="0"
+          iyy="1e-6" iyz="0"
+          izz="1e-6"
+      />
+    </inertial>
+    <collision name='collision'>
+      <origin xyz="0 0 0" rpy="0 0 0"/>
+      <geometry>
+        <box size=".01 .01 .01"/>
+      </geometry>
+    </collision>
+  </link>
+  <gazebo reference="scan_link_right">
+    <selfCollide>false</selfCollide>
+    <mu1 value="0.05" />
+    <mu2 value="0.05" />
+  </gazebo>
+   <!-- IMU -->
+  <joint name="imu_joint" type="fixed">
+    <origin xyz="0 0 0" rpy="0 0 0" />
+    <parent link="base_link"/>
+    <child link="imu_link" />
+  </joint>
+  <link name="imu_link">
+  </link>
+  <xacro:include filename="$(find lawn_robot_project)/description/robot.gazebo"/>
 </robot>

Commit message: Added IMU, EKF and nodes for autonomous movement, added utility node path_tacking

File: description/robot.urdf.xacro (robot description, xacro)
@@ -7,5 +7,5 @@
     <xacro:property name="Iy_body" value="{(1/12)*m1*(0.4*0.4+0.3*0.3)}"/>
     <xacro:property name="Iz_body" value="{(1/12)*m1*(0.4*0.4+0.2*0.2)}"/>
-    <xacro:property name="skid_mass" value="0.1"/> <!-- Mass of each skid -->
+    <xacro:property name="skid_mass" value="0.05"/> <!-- Mass of each skid -->
     <xacro:property name="skid_radius" value="0.02"/> <!-- Radius of the skid (capsule) -->
     <xacro:property name="skid_length" value="0.1"/> <!-- Length of the skid (capsule) -->
